File: Kaikuluotain_late_Eagle_tiedostot/Kaikuluotain_late.sch (EAGLE design)
At the start: 5 parts

Commit message: Valmis
Parts:
- added HYPPY5V: (no value), rcl:R-EU_0207/10
Connections:
- new net N$12: HYPPY5V.1, LCD1.VDD
- net 5V: now also HYPPY5V.2; no longer LCD1.VDD
- net GND: no longer U$1.GND1
Changed lines of the file:
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@@
 <setting verticaltext="up"/>
 </settings>
-<grid distance="0.1" unitdist="inch" unit="inch" style="lines" multiple="1" display="yes" altdistance="0.01" altunitdist="inch" altunit="inch"/>
+<grid distance="0.1" unitdist="inch" unit="inch" style="lines" multiple="1" display="no" altdistance="0.01" altunitdist="inch" altunit="inch"/>
 <layers>
 <layer number="1" name="Top" color="4" fill="1" visible="no" active="no"/>
@@
 </variantdefs>
 <classes>
-<class number="0" name="default" width="0" drill="0">
+<class number="0" name="default" width="0.762" drill="0.8">
+<clearance class="0" value="0.254"/>
 </class>
 </classes>
@@
 <part name="U$2" library="diy-modules" deviceset="ULTRASONIC-HC-SR04" device="#V"/>
 <part name="R1" library="resistor" library_urn="urn:adsk.eagle:library:348" deviceset="R-EU_" device="0411/15" package3d_urn="urn:adsk.eagle:package:23568/1" value="180"/>
+<part name="HYPPY5V" library="rcl" library_urn="urn:adsk.eagle:library:334" deviceset="R-EU_" device="0207/10" package3d_urn="urn:adsk.eagle:package:23491/1"/>
 </parts>
 <sheets>
@@
 <attribute name="VALUE" x="36.83" y="42.418" size="1.778" layer="96"/>
 </instance>
+<instance part="HYPPY5V" gate="G$1" x="48.26" y="78.74" smashed="yes">
+<attribute name="NAME" x="44.45" y="80.2386" size="1.778" layer="95"/>
+<attribute name="VALUE" x="44.45" y="75.438" size="1.778" layer="96"/>
+</instance>
 </instances>
 <busses>
@@
 </segment>
 <segment>
-<pinref part="LCD1" gate="G$1" pin="VDD"/>
-<wire x1="30.48" y1="78.74" x2="35.56" y2="78.74" width="0.1524" layer="91"/>
-<label x="33.02" y="78.74" size="1.778" layer="95"/>
-</segment>
-<segment>
 <pinref part="TRIM" gate="1" pin="E"/>
 <wire x1="45.72" y1="101.6" x2="50.8" y2="101.6" width="0.1524" layer="91"/>
 <label x="48.26" y="101.6" size="1.778" layer="95"/>
 </segment>
+<segment>
+<wire x1="53.34" y1="78.74" x2="60.96" y2="78.74" width="0.1524" layer="91"/>
+<label x="58.42" y="78.74" size="1.778" layer="95"/>
+<pinref part="HYPPY5V" gate="G$1" pin="2"/>
+</segment>
 </net>
 <net name="GND" class="0">
-<segment>
-<pinref part="U$1" gate="G$1" pin="GND1"/>
-<wire x1="96.52" y1="134.62" x2="96.52" y2="139.7" width="0.1524" layer="91"/>
-<label x="91.44" y="137.16" size="1.778" layer="95"/>
-</segment>
 <segment>
 <pinref part="U$2" gate="G$1" pin="GND"/>
@@
 <pinref part="U$1" gate="G$1" pin="D6"/>
 <wire x1="93.98" y1="68.58" x2="93.98" y2="73.66" width="0.1524" layer="91"/>
+</segment>
+</net>
+<net name="N$12" class="0">
+<segment>
+<pinref part="LCD1" gate="G$1" pin="VDD"/>
+<pinref part="HYPPY5V" gate="G$1" pin="1"/>
+<wire x1="30.48" y1="78.74" x2="43.18" y2="78.74" width="0.1524" layer="91"/>
 </segment>
 </net>
@@
 packages will not be understood (or retained) with this version.
 </note>
+<note version="8.4" severity="warning">
+Since Version 8.4, EAGLE supports properties for SPICE simulation.
+Probes in schematics and SPICE mapping objects found in parts and library devices
+will not be understood with this version. Update EAGLE to the latest version
+for full support of SPICE simulation.
+</note>
 </compatibility>
